File: 2025_04_STM32F103_RobotBrain/2025_04_STM32F103_RobotBrain.kicad_pcb (KiCad board)
At the start: 2 copper layers, 90 x 80 mm, 25 parts, among them J1 USB_B_Mini, SW1 SW_SPST, U1 STM32F103RCTx, U2 USBLC6-2SC6, Y2 16Mhz

Commit message: Robotbrain
Parts:
- added D4: Bl_IND_LED, LED_SMD:LED_0805_2012Metric, F.Cu at (197.1, 128.0)
- added J2: Conn_MPU6050, Connector_PinHeader_2.54mm:PinHeader_1x08_P2.54mm_Vertical, F.Cu at (161.1, 112.5)
- added J3: Conn_ULTRA, Connector_PinHeader_2.54mm:PinHeader_1x04_P2.54mm_Vertical, F.Cu at (206.0, 111.4)
- added J4: Conn_ULTRA, Connector_PinHeader_2.54mm:PinHeader_1x04_P2.54mm_Vertical, F.Cu at (200.9, 96.5)
- added J5: Conn_3V3, Connector_JST:JST_XH_B2B-XH-A_1x02_P2.50mm_Vertical, F.Cu at (192.6, 89.8)
- added J6: Conn_5V, Connector_JST:JST_XH_B2B-XH-A_1x02_P2.50mm_Vertical, F.Cu at (192.6, 97.5)
- added J7: Conn_DRIVE, Connector_JST:JST_XH_B4B-XH-A_1x04_P2.50mm_Vertical, F.Cu at (202.0, 89.8)
- added J8: Conn_HAL, Connector_JST:JST_XH_B5B-XH-A_1x05_P2.50mm_Vertical, F.Cu at (192.6, 82.0)
- added LED1: IN-PI55TATPRPGPB, RGB_LED:INPI55TATPRPGPB, F.Cu at (146.4, 115.8)
- added LED2: IN-PI55TATPRPGPB, RGB_LED:INPI55TATPRPGPB, F.Cu at (146.4, 123.8)
- added MDBT42T-AT1: MDBT42T-AT, MDBT42T-AT:MDBT42T, F.Cu at (182.0, 121.0)
- added Q1: BSS138, Package_TO_SOT_SMD:SOT-23, F.Cu at (153.1, 120.0)
- added R10: 10K, Resistor_SMD:R_0805_2012Metric_Pad1.20x1.40mm_HandSolder, F.Cu at (153.0, 116.1)
- added R7: 10K, Resistor_SMD:R_0805_2012Metric_Pad1.20x1.40mm_HandSolder, F.Cu at (197.2, 125.0)
- added R8: 10K, Resistor_SMD:R_0805_2012Metric_Pad1.20x1.40mm_HandSolder, F.Cu at (153.0, 113.2)
- added R9: 10K, Resistor_SMD:R_0805_2012Metric_Pad1.20x1.40mm_HandSolder, F.Cu at (205.6, 102.1)
- added SW2: SW_USER, Button_Switch_SMD:SW_SPST_PTS647_Sx50, F.Cu at (207.4, 97.4)
