File: Phase_B_Final_rev/2025_05_STM32F103_RobotBrain_LayoutComplete/2025_04_STM32F103_RobotBrain/2025_04_STM32F103_RobotBrain.kicad_pcb (KiCad board)
At the start: 2 copper layers, 90 x 80 mm, 47 parts, among them J1 USB_B_Mini, J10 CONN_TRACK, J11 CONN_UART, J2 CONN_MPU6050, J3 CONN_ULTRA, J4 CONN_SWD, J5 CONN_5V, J6 CONN_3V3, J7 CONN_DRIVE, J8 CONN_HAL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

Commit message: Robotbrain_final_rev
Routing:
- net /E2B: vias 4 -> 6
- net /E2A: vias 4 -> 8
- net +3V3: vias 9 -> 11
Changed lines of the file:
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@@
+	)
+	(segment
+		(start 166.5 51)
+		(end 166.5 55.5)
+		(width 0.254)
+		(layer "F.Cu")
+		(net 28)
 	)
 	(segment
@@
 	)
 	(via
+		(at 166.5 51)
+		(size 0.6)
+		(drill 0.3)
+		(layers "F.Cu" "B.Cu")
+		(net 28)
+	)
+	(via
 		(at 157.873 87)
 		(size 0.6)
@@
 	(via
 		(at 162 59)
+		(size 0.6)
+		(drill 0.3)
+		(layers "F.Cu" "B.Cu")
+		(net 28)
+	)
+	(via
+		(at 166.5 55.5)
 		(size 0.6)
 		(drill 0.3)
@@
 	)
 	(segment
-		(start 166.5 51)
-		(end 166.5 55.5)
-		(width 0.254)
-		(layer "B.Cu")
-		(net 28)
-	)
-	(segment
 		(start 145.465 70.335)
 		(end 145.11 70.69)
@@
 	)
 	(segment
+		(start 121.8895 94)
+		(end 117.5 94)
+		(width 0.254)
+		(layer "F.Cu")
+		(net 79)
+	)
+	(segment
+		(start 127.427 94)
+		(end 124.5 94)
+		(width 0.254)
+		(layer "F.Cu")
+		(net 79)
+	)
+	(segment
 		(start 104 83)
 		(end 104 80.5)
@@
 	)
 	(via
+		(at 124.5 94)
+		(size 0.6)
+		(drill 0.3)
+		(layers "F.Cu" "B.Cu")
+		(net 79)
+	)
+	(via
+		(at 127.427 94)
+		(size 0.6)
+		(drill 0.3)
+		(layers "F.Cu" "B.Cu")
+		(net 79)
+	)
+	(via
 		(at 104 80.5)
 		(size 0.6)
@@
 	)
 	(via
+		(at 117.5 94)
+		(size 0.6)
+		(drill 0.3)
+		(layers "F.Cu" "B.Cu")
+		(net 79)
+	)
+	(via
 		(at 113 91.5)
 		(size 0.6)
 		(drill 0.3)
 		(layers "F.Cu" "B.Cu")
+		(net 79)
+	)
+	(via
+		(at 121.8895 94)
+		(size 0.6)
+		(drill 0.3)
+		(layers "F.Cu" "B.Cu")
+		(net 79)
+	)
+	(segment
+		(start 117.5 94)
+		(end 115.5 94)
+		(width 0.254)
+		(layer "B.Cu")
+		(net 79)
+	)
+	(segment
+		(start 104 75.5)
+		(end 104.5 75)
+		(width 0.254)
+		(layer "B.Cu")
+		(net 79)
+	)
+	(segment
+		(start 104 80.5)
+		(end 104 75.5)
+		(width 0.254)
+		(layer "B.Cu")
+		(net 79)
+	)
+	(segment
+		(start 130 94)
+		(end 127.427 94)
+		(width 0.254)
+		(layer "B.Cu")
+		(net 79)
+	)
+	(segment
+		(start 124.5 94)
+		(end 121.8895 94)
+		(width 0.254)
+		(layer "B.Cu")
 		(net 79)
 	)
@@
 	)
 	(segment
-		(start 104 75.5)
-		(end 104.5 75)
-		(width 0.254)
-		(layer "B.Cu")
-		(net 79)
-	)
-	(segment
-		(start 104 80.5)
-		(end 104 75.5)
-		(width 0.254)
-		(layer "B.Cu")
-		(net 79)
-	)
-	(segment
-		(start 130 94)
-		(end 115.5 94)
-		(width 0.254)
-		(layer "B.Cu")
-		(net 79)
-	)
-	(segment
 		(start 115 83)
 		(end 110 78)
@@
 	)
 	(segment
+		(start 110 76)
+		(end 110 72.5)
+		(width 0.254)
+		(layer "F.Cu")
+		(net 80)
+	)
+	(segment
 		(start 139.57 97.57)
 		(end 130 88)
@@
 	)
 	(via
+		(at 110 76)
+		(size 0.6)
+		(drill 0.3)
+		(layers "F.Cu" "B.Cu")
+		(net 80)
+	)
+	(via
+		(at 110 72.5)
+		(size 0.6)
+		(drill 0.3)
+		(layers "F.Cu" "B.Cu")
+		(net 80)
+	)
+	(via
 		(at 130 86)
 		(size 0.6)
@@
 		(drill 0.3)
 		(layers "F.Cu" "B.Cu")
-		(net 80)
-	)
-	(segment
-		(start 110 78)
-		(end 110 70)
-		(width 0.254)
-		(layer "B.Cu")
 		(net 80)
 	)
@@
 	)
 	(segment
+		(start 110 72.5)
+		(end 110 70)
+		(width 0.254)
+		(layer "B.Cu")
+		(net 80)
+	)
+	(segment
 		(start 130 86)
 		(end 127 83)
 		(width 0.254)
 		(layer "B.Cu")
+		(net 80)
+	)
+	(segment
+		(start 110 78)
+		(end 110 76)
+		(width 0.254)
+		(layer "B.Cu")

Commit message: Robotbrain_final_rev
Routing:
- net +3V3: track 265.7 -> 273.3 mm
Other:
- board text added: "Embedded Systems Name : Ali Alalwia Version : 1.0 Date : 05/06/2025"
Changed lines of the file:
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@@
 		(allow_soldermask_bridges_in_footprints no)
 		(tenting front back)
+		(aux_axis_origin 92.1 109.750001)
+		(grid_origin 92.1 109.750001)
 		(pcbplotparams
 			(layerselection 0x00000000_00000000_55555555_5755f5ff)
@@
 			(outputformat 1)
 			(mirror no)
-			(drillshape 1)
+			(drillshape 0)
 			(scaleselection 1)
-			(outputdirectory "")
+			(outputdirectory "gerber/")
 		)
 	)
@@
 		)
 	)
+	(gr_text "Embedded Systems\nName : Ali Alalwia\nVersion : 1.0\nDate : 05/06/2025"
+		(at 95.6 37.750001 0)
+		(layer "F.SilkS")
+		(effects
+			(font
+				(size 1 1)
+				(thickness 0.2)
+				(bold yes)
+			)
+			(justify left bottom)
+		)
+	)
 	(gr_text "RGB 2"
 		(at 180.4 101.94 90)
@@
 	)
 	(segment
+		(start 98.72 46.27)
+		(end 94 50.99)
+		(width 0.381)
+		(layer "F.Cu")
+		(net 28)
+	)
+	(segment
 		(start 122.58 99.9)
 		(end 122.58 80.3275)
@@
 	)
 	(segment
-		(start 135.5775 60.34)
-		(end 135.5775 59.4575)
-		(width 0.254)
+		(start 94 75.25)
+		(end 97.51 78.76)
+		(width 0.381)
 		(layer "F.Cu")
 		(net 28)
@@
 	)
 	(segment
+		(start 94 50.99)
+		(end 94 75.25)
+		(width 0.381)
+		(layer "F.Cu")
+		(net 28)
+	)
+	(segment
 		(start 142.99 70.305)
 		(end 142.52 69.835)
@@
 		(width 0.254)
 		(layer "F.Cu")
-		(net 28)
-	)
-	(segment
-		(start 135.5775 59.4575)
-		(end 116.16 40.04)
-		(width 0.254)
-		(layer "F.Cu")

Commit message: Robotbrain_final_rev
Routing:
- net +3V3: track 273.3 -> 358.7 mm, vias 11 -> 13
- net /PS2_CS: track 48.8 -> 50.6 mm
- net GND: vias 44 -> 56
